File: pcb/heater-controller.kicad_pcb (KiCad board)
At the start: 2 copper layers, 125 x 99.9 mm, 58 parts, among them J2 Conn_01x08_Socket, Q1 100V/1.3mR, Q10 80V/790uR, Q11 80V/790uR, Q12 80V/790uR, Q13 80V/790uR, Q14 80V/790uR, Q2 100V/1.3mR, Q3 100V/1.3mR, Q4 100V/1.3mR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

Commit message: Update sch & pcb
Parts:
- removed C6, C7: 100n, Capacitor_SMD:C_0603_1608Metric
- removed H5, H6, H7: M4, MountingHole:MountingHole_6.4mm_M6_Pad_Via
- removed U6, U7: IX4310T, Package_TO_SOT_SMD:SOT-23-5_HandSoldering
- added C11: 1u/100V, Capacitor_SMD:C_1210_3225Metric, F.Cu at (61.4, 93.2)
- added J1: Conn_01x03_Socket, Connector_PinHeader_2.54mm:PinHeader_1x04_P2.54mm_Vertical, F.Cu at (77.0, 3.00)
- added J3: Conn_01x03_Socket, Connector_PinHeader_2.54mm:PinHeader_1x04_P2.54mm_Vertical, F.Cu at (95.5, 3.00)
- added J4: Conn_01x03_Socket, Connector_PinHeader_2.54mm:PinHeader_1x04_P2.54mm_Vertical, F.Cu at (41.0, 3.00)
- added R19: 10k, Resistor_SMD:R_0603_1608Metric, F.Cu at (101.6, 3.00)
- added RV1: 100k, Potentiometer_THT:Potentiometer_Bourns_3296Y_Vertical, F.Cu at (7.74, 40.3)
- added RV2: 100k, Potentiometer_THT:Potentiometer_Bourns_3296Y_Vertical, F.Cu at (1.72, 31.1)
- added TVS2: 64V, Diode_SMD:D_SMC, F.Cu at (50.8, 94.0)
- added TVS3: 64V, Diode_SMD:D_SMC, F.Cu at (97.6, 94.8)
- added TVS4: 64V, Diode_SMD:D_SMC, F.Cu at (97.4, 63.6)
- added TVS5: 64V, Diode_SMD:D_SMC, F.Cu at (97.4, 33.0)
- H10, H8, H9: footprint MountingHole:MountingHole_6.4mm_M6_Pad_Via -> connectors:KEYS_7798
- R16: value 10k -> 180k
- U1: value IX4310T -> TMP390; footprint Package_TO_SOT_SMD:SOT-23-5_HandSoldering -> Package_TO_SOT_SMD:SOT-666
- moved R16 93.5 mm to (10.6, 73.4), turned to -90 degrees
- moved C1 92.7 mm to (12.4, 75.8)
- moved U1 92.1 mm to (13.2, 73.6)
- moved R17 47.4 mm to (98.4, 3.00), turned to 90 degrees
- moved TVS1 47.1 mm to (52.0, 3.60), turned to 0 degrees
- moved R18 29.2 mm to (100.0, 3.00), turned to 90 degrees
- moved C2 6.68 mm to (61.4, 4.20), turned to 90 degrees
- moved Q11 6.00 mm to (96.0, 42.0)
- moved Q12 6.00 mm to (96.0, 54.0)
- moved Q10 4.00 mm to (96.0, 73.0)
- moved Q9 4.00 mm to (96.0, 85.0)
- moved U2 3.61 mm to (13.8, 42.6), turned to -90 degrees
- moved H8 3.00 mm to (111.0, 72.0)
- moved H10 2.00 mm to (111.0, 21.0)
- moved C3 1.61 mm to (11.2, 42.6), turned to 90 degrees
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Connections:
- net Net-(U4-Vbus) renamed +60V_OUT
- C1 pad 1: +12V -> +3V3
- C2 pad 2: GNDD -> PGND
- H1 pad 1: Earth -> unconnected-(H1-Pad1)_6
- H2 pad 1: Earth -> unconnected-(H2-Pad1)_7
- H3 pad 1: Earth -> unconnected-(H3-Pad1)_8
- H4 pad 1: Earth -> unconnected-(H4-Pad1)
- Q10 pad 1: Net-(Q10-G) -> Net-(J3-Pin_1)
- Q10 pad 2: GNDD -> PGND
- Q11 pad 1: Net-(Q11-G) -> Net-(J3-Pin_2)
- Q11 pad 2: GNDD -> PGND
- Q12 pad 1: Net-(Q11-G) -> Net-(J3-Pin_2)
- Q12 pad 2: GNDD -> PGND
- Q13 pad 2: GNDD -> PGND
- Q14 pad 2: GNDD -> PGND
- Q9 pad 1: Net-(Q10-G) -> Net-(J3-Pin_1)
- Q9 pad 2: GNDD -> PGND
- R14 pad 1: Net-(U2-EN/UVLO) -> Net-(U1-~{OUTA})
- R16 pad 1: DRV1 -> Net-(U1-SETA)
- R17 pad 1: DRV1 -> Net-(J3-Pin_1)
- R17 pad 2: GNDD -> PGND
- R18 pad 1: DRV1 -> Net-(J3-Pin_2)
- R18 pad 2: GNDD -> PGND
- TVS1 pad 2: Earth -> PGND
- U1 pad 1: DRV1 -> Net-(U1-SETA)
- U1 pad 3: Net-(Q10-G) -> GNDD
- U1 pad 4: Net-(Q10-G) -> unconnected-(U1-~{OUTB}-Pad4)
- U1 pad 5: +12V -> +3V3
- U2 pad 1: Net-(U2-EN/UVLO) -> Net-(U1-~{OUTA})
- U3 pad 3: Net-(U2-EN/UVLO) -> Net-(U1-~{OUTA})
Routing:
- net Net-(J3-Pin_1): track 0.00 -> 85.2 mm, vias 0 -> 2
- net Net-(U1-~{OUTA}): track 0.00 -> 75.3 mm, vias 0 -> 4
- net Net-(J3-Pin_2): track 0.00 -> 57.5 mm, vias 0 -> 2
- net Net-(U2-EN/UVLO): track 33.1 -> 0.00 mm
- net Net-(Q2-D): track 26.4 -> 58.0 mm, vias 0 -> 120
- net Net-(J3-Pin_3): track 0.00 -> 31.2 mm, vias 0 -> 2
- net +60V: track 18.3 -> 45.1 mm, vias 1 -> 142
- net Net-(U2-OV): track 6.18 -> 21.0 mm, vias 0 -> 1
- net PGND: track 0.00 -> 14.5 mm, vias 0 -> 183
- net Net-(Q1-G): track 123.0 -> 108.6 mm
- net Net-(R13-Pad2): track 34.3 -> 28.4 mm, vias 0 -> 2
- net +3V3: track 36.0 -> 41.5 mm
- net Net-(Q1-S): track 7.03 -> 3.12 mm, vias 0 -> 128
- net Net-(Q10-G): track 2.70 -> 0.00 mm
- net Net-(U1-SETA): track 0.00 -> 1.95 mm
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- added copper zone on B.Cu, net +60V
- added copper zone on B.Cu, net +60V_OUT
- added copper zone on B.Cu, net HEATER1
- added copper zone on B.Cu, net HEATER2
- added copper zone on B.Cu, net HEATER3
- added copper zone on B.Cu, net Net-(Q1-S)
- added copper zone on B.Cu, net Net-(Q2-D)
- added copper zone on B.Cu, net PGND
- added copper zone on F.Cu, net PGND
- removed copper zone on F.Cu, net GNDD
Other:
- board size 125 x 99.9 mm -> 125 x 99.8 mm
- board text added: "HEAT1-OUT"
- board text added: "HEAT2-OUT"
- board text added: "HEAT3-OUT"
