File: pcb/heater.kicad_sch (KiCad schematic)
At the start: 19 parts, among them Q10 80V/790uR, Q11 80V/790uR, Q12 80V/790uR, Q13 80V/790uR, Q14 80V/790uR, Q9 80V/790uR, U1 IX4310T, U6 IX4310T, U7 IX4310T

Commit message: Update sch & pcb
Parts:
- removed C1, C6, C7: 100n, Capacitor_SMD:C_0603_1608Metric, symbol Device:C_Small
- removed H7: M4, MountingHole:MountingHole_6.4mm_M6_Pad_Via, symbol Mechanical:MountingHole_Pad
- removed R16: 10k, Resistor_SMD:R_0603_1608Metric, symbol Device:R_Small
- removed U1, U6, U7: IX4310T, Package_TO_SOT_SMD:SOT-23-5_HandSoldering, symbol drivers:GATE_DRV_IN_OUT_OUT
- added J3: Conn_01x03_Socket, Connector_PinHeader_2.54mm:PinHeader_1x04_P2.54mm_Vertical, symbol Connector:Conn_01x04_Socket
- added R19: 10k, Resistor_SMD:R_0603_1608Metric, symbol Device:R_Small
- added TVS3, TVS4, TVS5: 64V, Diode_SMD:D_SMC, symbol passives:d_tvs_bidi
- H10, H8, H9: footprint MountingHole:MountingHole_6.4mm_M6_Pad_Via -> connectors:KEYS_7798
Connections:
- net HEATER1: now also TVS3.1 (K)
- net HEATER2: now also TVS4.1 (K)
- net HEATER3: now also TVS5.1 (K)
- net at Q13.1 (G), Q14.1 (G): now also J3.3 (Pin_3), R19.1
- net at Q10.1 (G), Q9.1 (G): now also R17.1, J3.1 (Pin_1)
- net at Q11.1 (G), Q12.1 (G): now also R18.1, J3.2 (Pin_2)
- removed net DRV1: R17.1, R18.1
- net GNDD renamed PGND
- net PGND: now also J3.4 (Pin_4), R19.2, TVS3.2 (A), TVS4.2 (A), TVS5.2 (A)
Other:
- moved on the sheet: H10, H8, H9, Q10, Q11, Q12, Q13, Q14, Q9
