File: pcb/power.kicad_sch (KiCad schematic)
At the start: 37 parts, among them J2 Conn_01x08_Socket, Q1 100V/1.3mR, Q2 100V/1.3mR, Q3 100V/1.3mR, Q4 100V/1.3mR, Q5 100V/1.3mR, Q6 100V/1.3mR, Q7 100V/1.3mR, Q8 100V/1.3mR, U2 LM74502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

Commit message: Update sch & pcb
Parts:
- removed H5, H6: M4, MountingHole:MountingHole_6.4mm_M6_Pad_Via, symbol Mechanical:MountingHole_Pad
- added C1: 100n, Capacitor_SMD:C_0603_1608Metric, symbol Device:C_Small
- added C11: 1u/100V, Capacitor_SMD:C_1210_3225Metric, symbol Device:C_Small
- added J1, J4: Conn_01x03_Socket, Connector_PinHeader_2.54mm:PinHeader_1x04_P2.54mm_Vertical, symbol Connector:Conn_01x04_Socket
- added R16: 180k, Resistor_SMD:R_0603_1608Metric, symbol Device:R_Small
- added TVS2: 64V, Diode_SMD:D_SMC, symbol passives:d_tvs_bidi
- added U1: TMP390, Package_TO_SOT_SMD:SOT-666, symbol sensors:TMP390
- RV1, RV2: footprint (none) -> Potentiometer_THT:Potentiometer_Bourns_3296Y_Vertical
Connections:
- net +3V3: now also C1.1, U1.5 (VDD)
- net +60V: now also J4.1 (Pin_1), J4.2 (Pin_2), J4.3 (Pin_3), J4.4 (Pin_4)
- net GNDD: now also C1.2, R16.2, U1.2 (SETB), U1.3 (GND); no longer C2.2
- net at R14.1, RV2.1, RV2.2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: now also U1.6 (~{OUTA})
- net +60V_OUT: now reaches R1.1, R10.1, R11.1, R3.1, R6.1, R7.1, R8.1, R9.1, U4.8 (Vbus), U4.9 (Vin-)
- net +60V_OUT: now also C11.1, TVS2.1 (K)
- net Earth renamed PGND
- net PGND: now also C2.2, C11.2, J1.1 (Pin_1), J1.2 (Pin_2), J1.3 (Pin_3), J1.4 (Pin_4), TVS2.2 (A)
- new net: R16.1, U1.1 (SETA)
- no-connect marks 2 -> 5
Other:
- note added: "Note: Trip point 102°C, hysteresis 20°C, release 82°C"
- moved on the sheet: C2, C3, C4, C5, Q1, Q2, Q3, Q4, Q5, Q6, Q7, Q8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
